File: eagle/SQR_FG_Digital.brd (EAGLE design)
At the start: 91.1 x 55.9 mm, 25 parts, among them IC1 MEGA328P, IC3 7805T, Q1 16MHz

Commit message: SQR_FG_Digital: I2Cの信号をピンソケットで出力できるように変更
Parts:
- added JP8: I2C-OUT, pinhead:1X02
- moved C12 5.08 mm to (59.7, 40.6)
- moved C13 5.08 mm to (54.6, 40.6)
Connections:
- net +3V3: now also C14.+, JP5.3; no longer JP5.5
- net +5V: now also JP5.5; no longer C14.+, JP5.3
- net GND: no longer IC1.21
- net SCL: now also JP8.1
- net SDA: now also JP8.2
Routing:
- net +3V3: track 43.2 -> 62.0 mm
- net +5V: track 175.3 -> 167.6 mm
Changed lines of the file:
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@@
 <element name="C10" library="rcl" package="TT2D5L" value="47uF" x="38.1" y="11.43" rot="MR270"/>
 <element name="C11" library="rcl" package="TT2D5L" value="47uF" x="48.26" y="8.89" rot="R270"/>
-<element name="C12" library="rcl" package="C025-024X044" value="0.1uF" x="54.61" y="40.64" rot="R180"/>
-<element name="C13" library="rcl" package="C025-024X044" value="0.1uF" x="59.69" y="40.64" rot="R180"/>
+<element name="C12" library="rcl" package="C025-024X044" value="0.1uF" x="59.69" y="40.64" rot="R180"/>
+<element name="C13" library="rcl" package="C025-024X044" value="0.1uF" x="54.61" y="40.64" rot="R180"/>
 <element name="C14" library="rcl" package="TT2D5L" value="47uF" x="48.26" y="44.45" rot="R90"/>
 <element name="C2" library="rcl" package="C050-024X044" value="22pF" x="10.16" y="17.78"/>
@@
 <element name="JP7" library="pinhead" package="1X02" value="5V" x="49.53" y="5.08" rot="R180"/>
 <element name="JP2" library="pinhead" package="1X04" value="DIGITAL_OUT" x="26.67" y="5.08"/>
+<element name="JP8" library="pinhead" package="1X02" value="I2C-OUT" x="25.4" y="44.45" rot="R270"/>
 </elements>
 <signals>
@@
 <contactref element="IC3" pad="2"/>
 <contactref element="JP6" pad="2"/>
-<contactref element="C12" pad="2"/>
 <contactref element="C13" pad="2"/>
 <contactref element="C14" pad="-"/>
 <contactref element="JP5" pad="1"/>
 <contactref element="JP1" pad="8"/>
-<contactref element="IC1" pad="21"/>
 <contactref element="JP7" pad="2"/>
 <wire x1="5.08" y1="10.16" x2="5.08" y2="17.78" width="0.4064" layer="16"/>
@@
 <wire x1="17.78" y1="27.94" x2="17.78" y2="10.16" width="0.4064" layer="16"/>
 <wire x1="17.78" y1="10.16" x2="5.08" y2="10.16" width="0.4064" layer="16"/>
-<wire x1="22.86" y1="27.94" x2="15.24" y2="27.94" width="0.4064" layer="16"/>
-<wire x1="22.86" y1="27.94" x2="22.86" y2="30.48" width="0.4064" layer="16"/>
-<wire x1="22.86" y1="27.94" x2="25.4" y2="27.94" width="0.4064" layer="16"/>
 <wire x1="22.86" y1="30.48" x2="20.32" y2="30.48" width="0.4064" layer="16"/>
 <wire x1="20.32" y1="30.48" x2="20.32" y2="48.26" width="0.4064" layer="16"/>
@@
 <wire x1="35.56" y1="20.32" x2="35.56" y2="17.78" width="0.4064" layer="16"/>
 <wire x1="55.88" y1="27.94" x2="35.56" y2="27.94" width="0.4064" layer="16"/>
-<wire x1="48.26" y1="45.72" x2="50.8" y2="45.72" width="0.4064" layer="16"/>
-<wire x1="50.8" y1="45.72" x2="50.8" y2="43.18" width="0.4064" layer="16"/>
 <contactref element="JP5" pad="2"/>
 <contactref element="JP5" pad="4"/>
-<wire x1="58.42" y1="40.64" x2="58.42" y2="43.18" width="0.4064" layer="16"/>
-<wire x1="53.34" y1="40.64" x2="53.34" y2="43.18" width="0.4064" layer="16"/>
-<wire x1="53.34" y1="43.18" x2="53.34" y2="45.72" width="0.4064" layer="16"/>
-<wire x1="53.34" y1="45.72" x2="58.42" y2="45.72" width="0.4064" layer="16"/>
-<wire x1="58.42" y1="45.72" x2="58.42" y2="43.18" width="0.4064" layer="16"/>
-<wire x1="50.8" y1="45.72" x2="53.34" y2="45.72" width="0.4064" layer="16"/>
 <wire x1="68.58" y1="33.02" x2="71.12" y2="33.02" width="0.4064" layer="16"/>
 <wire x1="71.12" y1="33.02" x2="71.12" y2="45.72" width="0.4064" layer="16"/>
 <wire x1="71.12" y1="45.72" x2="58.42" y2="45.72" width="0.4064" layer="16"/>
+<wire x1="58.42" y1="45.72" x2="53.34" y2="45.72" width="0.4064" layer="16"/>
+<wire x1="53.34" y1="45.72" x2="48.26" y2="45.72" width="0.4064" layer="16"/>
 <wire x1="68.58" y1="22.86" x2="71.12" y2="22.86" width="0.4064" layer="16"/>
 <wire x1="71.12" y1="22.86" x2="71.12" y2="33.02" width="0.4064" layer="16"/>
@@
 <wire x1="55.88" y1="22.86" x2="68.58" y2="22.86" width="0.4064" layer="16"/>
 <wire x1="7.62" y1="17.78" x2="5.08" y2="17.78" width="0.4064" layer="16"/>
+<contactref element="C12" pad="2"/>
+<wire x1="48.26" y1="45.72" x2="50.8" y2="45.72" width="0.4064" layer="16"/>
+<wire x1="50.8" y1="45.72" x2="50.8" y2="43.18" width="0.4064" layer="16"/>
+<wire x1="53.34" y1="43.18" x2="53.34" y2="45.72" width="0.4064" layer="16"/>
+<wire x1="58.42" y1="43.18" x2="58.42" y2="45.72" width="0.4064" layer="16"/>
+<wire x1="58.42" y1="40.64" x2="58.42" y2="43.18" width="0.4064" layer="16"/>
+<wire x1="53.34" y1="40.64" x2="53.34" y2="43.18" width="0.4064" layer="16"/>
+<wire x1="25.4" y1="27.94" x2="25.4" y2="30.48" width="0.4064" layer="16"/>
+<wire x1="25.4" y1="30.48" x2="22.86" y2="30.48" width="0.4064" layer="16"/>
+<wire x1="17.78" y1="27.94" x2="20.32" y2="27.94" width="0.4064" layer="16"/>
+<wire x1="20.32" y1="27.94" x2="20.32" y2="30.48" width="0.4064" layer="16"/>
 </signal>
 <signal name="N$3">
@@
 <contactref element="C11" pad="+"/>
 <contactref element="C9" pad="1"/>
-<contactref element="C12" pad="1"/>
-<contactref element="C14" pad="+"/>
-<contactref element="JP5" pad="3"/>
 <contactref element="R2" pad="1"/>
 <contactref element="JP7" pad="1"/>
@@
 <wire x1="50.8" y1="5.08" x2="50.8" y2="10.16" width="0.4064" layer="16"/>
 <wire x1="50.8" y1="10.16" x2="48.26" y2="10.16" width="0.4064" layer="16"/>
-<wire x1="55.88" y1="43.18" x2="55.88" y2="40.64" width="0.4064" layer="16"/>
-<wire x1="55.88" y1="35.56" x2="55.88" y2="38.1" width="0.4064" layer="16"/>
-<wire x1="55.88" y1="38.1" x2="55.88" y2="40.64" width="0.4064" layer="16"/>
-<wire x1="48.26" y1="43.18" x2="48.26" y2="38.1" width="0.4064" layer="16"/>
-<wire x1="48.26" y1="38.1" x2="55.88" y2="38.1" width="0.4064" layer="16"/>
 <wire x1="50.8" y1="12.7" x2="50.8" y2="10.16" width="0.4064" layer="16"/>
 <wire x1="45.72" y1="15.24" x2="50.8" y2="15.24" width="0.4064" layer="1"/>
@@
 <wire x1="20.32" y1="2.54" x2="50.8" y2="2.54" width="0.4064" layer="16"/>
 <wire x1="50.8" y1="2.54" x2="50.8" y2="5.08" width="0.4064" layer="16"/>
+<contactref element="JP5" pad="5"/>
+<contactref element="C12" pad="1"/>
+<wire x1="60.96" y1="40.64" x2="60.96" y2="43.18" width="0.4064" layer="16"/>
+<wire x1="55.88" y1="35.56" x2="60.96" y2="35.56" width="0.4064" layer="16"/>
+<wire x1="60.96" y1="35.56" x2="60.96" y2="40.64" width="0.4064" layer="16"/>
 </signal>
 <signal name="SDA">
 <contactref element="IC1" pad="27"/>
 <contactref element="JP1" pad="5"/>
-<wire x1="22.86" y1="43.18" x2="30.48" y2="43.18" width="0.4064" layer="16"/>
 <wire x1="30.48" y1="43.18" x2="30.48" y2="33.02" width="0.4064" layer="16"/>
 <wire x1="30.48" y1="33.02" x2="58.42" y2="33.02" width="0.4064" layer="16"/>
 <wire x1="58.42" y1="33.02" x2="58.42" y2="25.4" width="0.4064" layer="16"/>
 <wire x1="58.42" y1="25.4" x2="68.58" y2="25.4" width="0.4064" layer="16"/>
+<contactref element="JP8" pad="2"/>
+<wire x1="22.86" y1="43.18" x2="25.4" y2="43.18" width="0.4064" layer="16"/>
+<wire x1="25.4" y1="43.18" x2="30.48" y2="43.18" width="0.4064" layer="16"/>
 </signal>
 <signal name="SCL">
@@
 <wire x1="66.04" y1="36.83" x2="33.02" y2="36.83" width="0.4064" layer="1"/>
 <wire x1="33.02" y1="36.83" x2="33.02" y2="45.72" width="0.4064" layer="1"/>
-<wire x1="33.02" y1="45.72" x2="22.86" y2="45.72" width="0.4064" layer="1"/>
+<contactref element="JP8" pad="1"/>
+<wire x1="22.86" y1="45.72" x2="25.4" y2="45.72" width="0.4064" layer="16"/>
+<wire x1="25.4" y1="45.72" x2="33.02" y2="45.72" width="0.4064" layer="1"/>
 </signal>
 <signal name="+3V3">
 <contactref element="JP1" pad="1"/>
 <contactref element="C13" pad="1"/>
-<contactref element="JP5" pad="5"/>
-<wire x1="60.96" y1="43.18" x2="60.96" y2="40.64" width="0.4064" layer="16"/>
-<wire x1="60.96" y1="40.64" x2="72.39" y2="40.64" width="0.4064" layer="1"/>
-<wire x1="72.39" y1="40.64" x2="72.39" y2="15.24" width="0.4064" layer="1"/>
-<wire x1="72.39" y1="15.24" x2="68.58" y2="15.24" width="0.4064" layer="1"/>
+<contactref element="JP5" pad="3"/>
+<contactref element="C14" pad="+"/>
+<wire x1="48.26" y1="43.18" x2="48.26" y2="38.1" width="0.4064" layer="16"/>
+<wire x1="48.26" y1="38.1" x2="55.88" y2="38.1" width="0.4064" layer="16"/>
+<wire x1="55.88" y1="38.1" x2="55.88" y2="40.64" width="0.4064" layer="16"/>
+<wire x1="55.88" y1="40.64" x2="55.88" y2="43.18" width="0.4064" layer="16"/>
+<wire x1="68.58" y1="15.24" x2="72.39" y2="15.24" width="0.4064" layer="1"/>
+<wire x1="72.39" y1="15.24" x2="72.39" y2="38.1" width="0.4064" layer="1"/>
+<wire x1="72.39" y1="38.1" x2="58.42" y2="38.1" width="0.4064" layer="1"/>
+<wire x1="58.42" y1="38.1" x2="55.88" y2="40.64" width="0.4064" layer="1"/>
 </signal>
 <signal name="RST">
@@
 </signal>
 </signals>
+<errors>
+</errors>
 </board>
 </drawing>

Commit message: SQR_FG_Digital.sch: LCDのRST信号の分圧抵抗を変更
Parts:
- R5: value 10k -> 47k
Changed lines of the file:
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@@
 <element name="R1" library="rcl" package="0207/10" value="10k" x="12.7" y="40.64" rot="R90"/>
 <element name="R4" library="rcl" package="0207/7" value="22k" x="59.69" y="30.48"/>
-<element name="R5" library="rcl" package="0207/7" value="10k" x="59.69" y="27.94" rot="R180"/>
+<element name="R5" library="rcl" package="0207/7" value="47k" x="59.69" y="27.94" rot="R180"/>
 <element name="JP5" library="pinhead" package="1X05" value="TLV1117-33" x="55.88" y="43.18"/>
 <element name="R2" library="rcl" package="0207/7" value="1k" x="59.69" y="35.56"/>
