File: eagle/SQR_FG_Digital.sch (EAGLE design)
At the start: 35 parts, among them IC1 MEGA328P, IC2 NJM7032, IC3 7805T, IC4 TLV1117-33, Q1 16MHz, T1 2SK4017, T2 2SK4017

Commit message: eagle files: デジタル部と出力部に基板を分割
Parts:
- removed C3, C7: 100uF, rcl:CPOL-EUE2.5-5
- removed C5: 0.1uF, rcl:C-EU025-024X044
- removed C6: 22pF, rcl:C-EU025-024X044
- removed IC2: NJM7032, linear:LM358N
- removed IC4: TLV1117-33, ic-package:DIL10
- removed R3, R7, R8: 10k, rcl:R-EU_0207/7
- removed R6: 10, rcl:R-EU_0207/7
- removed T1, T2: 2SK4017, zetex:NMOSE3L
- added JP7: 5V, pinhead:PINHD-1X2
- added R2: 1k, rcl:R-EU_0207/7
- C1, C2: device rcl:C-EU025-024X044 -> rcl:C-EU050-024X044
- JP2: value OUT -> DIGITAL_OUT; device pinhead:PINHD-1X2 -> pinhead:PINHD-1X4
- JP4: value Encoder -> ENCODER
- JP5: value Level -> TLV1117-33; device pinhead:PINHD-1X3 -> pinhead:PINHD-1X5
- R1: device rcl:R-EU_0207/7 -> rcl:R-EU_0207/10
- R5: value 12k -> 10k
Connections:
- removed net AGND: C5.2, C6.1, C7.-, IC2P.V-, R8.1, T2.S
- removed net N$11: JP2.1, R6.2
- removed net N$15: C6.2, IC2A.+IN, JP5.2
- removed net N$16: IC2A.-IN, IC2A.OUT, R6.1
- removed net N$17: C3.-, C7.+, IC2B.+IN, R7.1, R8.2
- removed net N$8: JP5.1, R3.1
- removed net VGND: IC2B.-IN, IC2B.OUT, T1.S
- new net N$5: C10.+, C8.1, D1.C, IC3.VI, JP6.1
- new net OC1A: IC1.PB1(OC1A), JP2.1
- net +3V3: now also JP5.5; no longer IC4.5
- net +5V: now also D1.A, JP5.3, JP7.1, R2.1; no longer C10.+, C3.+, C5.1, C8.1, IC2P.V+, IC3.VI, IC4.3, JP6.1, R7.2
- net GND: now also IC1.AREF, JP1.8, JP5.1, JP5.2, JP5.4, JP7.2; no longer IC4.1
- net N$6: now also JP1.9, R2.2; no longer JP2.2, JP5.3, T1.D, T2.D
- net SW_GND: now also JP2.3; no longer T2.G
- net SW_VGND: now also JP2.4; no longer T1.G
- net WAVE_OUT: now also JP2.2; no longer R3.2
Other:
- moved on the sheet: C1, C10, C11, C12, C13, C14, C2, C4, C8, C9, D1, IC1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

Commit message: SQR_FG_Digital: I2Cの信号をピンソケットで出力できるように変更
Parts:
- added JP8: I2C-OUT, pinhead:PINHD-1X2
Connections:
- net +3V3: now also C14.+, JP5.3; no longer JP5.5
- net +5V: now also JP5.5; no longer C14.+, JP5.3
- net GND: no longer IC1.AREF
- net SCL: now also JP8.1
- net SDA: now also JP8.2
Other:
- moved on the sheet: C12, C13, C14, JP1, JP5

Commit message: SQR_FG_Digital.sch: LCDのRST信号の分圧抵抗を変更
Parts:
- R5: value 10k -> 47k
Changed lines of the file:
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@@
 <part name="C4" library="rcl" deviceset="C-EU" device="025-024X044" value="0.1uF"/>
 <part name="R4" library="rcl" deviceset="R-EU_" device="0207/7" value="22k"/>
-<part name="R5" library="rcl" deviceset="R-EU_" device="0207/7" value="10k"/>
+<part name="R5" library="rcl" deviceset="R-EU_" device="0207/7" value="47k"/>
 <part name="GND5" library="supply1" deviceset="GND" device=""/>
 <part name="JP3" library="pinhead" deviceset="PINHD-1X3" device="" value="Duty"/>
